File: Starbie.kicad_pcb (KiCad board)
At the start: 2 copper layers, 98.6 x 103.2 mm, 7 parts, among them J1 Conn_01x04_Pin, J2 Conn_01x08_Pin, SW1 SW_Push, SW2 SW_Push, U1 XIAO-ESP32-C3-SMD, U2 DHT11

Commit message: I FIXED THE WIRES and added my chud star pet
Routing:
- net GND: track 26.7 -> 203.5 mm
- net /GPIO2: track 0.00 -> 68.1 mm
- net /SCL: track 0.00 -> 60.6 mm
- net /SDA: track 0.00 -> 60.2 mm
- net +3.3V: track 141.6 -> 198.0 mm
- net /GPIO3: track 50.8 -> 54.2 mm
Other:
- board size 98.6 x 103.2 mm -> 99.2 x 103.2 mm
